Commit message: first commit

File: cubli_description/urdf/cubli.xacro (robot description, xacro)
@@ -32,11 +32,4 @@
         <box size="${cube_length} ${cube_length} ${cube_length}" />
       </geometry>
-      <material>
-        <script>
-          <uri>model://mud_box/materials/scripts</uri>
-          <uri>model://mud_box/materials/textures</uri>
-          <name>vrc/mud</name>
-        </script>
-      </material>
     </visual>
     <collision>
